File: 500mA_7Chan/teensy3x_solenoid_driver.sch (KiCad schematic (older format))
At the start: 11 parts, among them J1 Conn_01x02, J2 Conn_01x02, J3 Conn_01x02, J4 Conn_01x02, J5 Conn_01x02, J6 Conn_01x02, J7 Conn_01x02, J8 Conn_02x05_Odd_Even, J9 Jack-DC, U1 TEENSY3x, U2 TBD62003A

Commit message: Finished initial layout and routing for 500mA design.
Parts:
- added C1: 10uF, Capacitor_SMD:C_0805_2012Metric, symbol Device:C
- J1, J2, J3, J4, J5, J6, J7: footprint (none) -> Connector_JST:JST_PH_S2B-PH-K_1x02_P2.00mm_Horizontal
- J8: footprint (none) -> 5x2_shrd_header:5X2_SHRD_HEADER
- J9: footprint (none) -> Connector_BarrelJack:BarrelJack_CUI_PJ-063AH_Horizontal
- U1: footprint (none) -> teensy3x:TEENSY3X
- U2: footprint (none) -> SOP-16_custom:SOP-16_3.9x9.9mm_P1.27mm
Connections:
- wire segments 78 -> 81
Other:
- note added: "LSCS# C440198"
- moved on the sheet: J1, J2, J3, J4, J5, J6, J7, J8, J9, U1

Commit message: Added finished initial design of 7channel driver.
Parts:
- added D1, D2, D3, D4, D5, D6, D7: LED_ALT, LED_SMD:LED_0603_1608Metric, symbol Device:LED_ALT
- added R1, R2, R3, R4, R5, R6, R7: 120, Resistor_SMD:R_0603_1608Metric, symbol Device:R
- C1: footprint Capacitor_SMD:C_0805_2012Metric -> LED_SMD:LED_0603_1608Metric
Connections:
- wire segments 81 -> 109
Other:
- note added: "Blue LED LCSC# C72041\nResistor LCSC# C22787"
- moved on the sheet: C1, J1, J2, J3, J4, J5, J6, J7, J8, J9, U1
